Commit message: Nandalal: URDF file chenged with new code

File: simulation/ros2_ws/src/cobot_sim/urdf/cobot.urdf.xacro (robot description, xacro)
@@ -1,14 +1,54 @@
-<?xml version="1.0">
-<robot name = "cobot" xmlns : xacro= "http://www.ros.org/wiki/xacro">
-  <link name = "base_link">
-    <visual><geometry><cylinder radius="0.2" length="0.15"/></geometry></visual>
-    <collision><geometry><cylinder radius="0.2" length="0.15"/></geometry></collision>
-    <inertial><mass value="5"/>
-      <inertia ixx="0.1" iyy="0.1" izz="0.1" ixy="0" iyz="0" ixz="0" />
+<?xml version="1.0"?>
+<robot name="cobot" xmlns:xacro="http://www.ros.org/wiki/xacro">
+  <link name="base_link">
+    <visual>
+      <geometry><cylinder radius="0.2" length="0.15"/></geometry>
+    </visual>
+    <collision>
+      <geometry><cylinder radius="0.2" length="0.15"/></geometry>
+    </collision>
+    <inertial>
+      <mass value="5"/>
+      <inertia ixx="0.1" iyy="0.1" izz="0.1" ixy="0" ixz="0" iyz="0"/>
     </inertial>
   </link>
-  <!-- Differential Drive plugin: responding to /cmd_vel, publishes /odom -->
+  <link name="left_wheel">
+    <visual>
+      <geometry><cylinder radius="0.05" length="0.04"/></geometry>
+    </visual>
+    <collision>
+      <geometry><cylinder radius="0.05" length="0.04"/></geometry>
+    </collision>
+    <inertial>
+      <mass value="0.5"/>
+      <inertia ixx="0.001" iyy="0.001" izz="0.001" ixy="0" ixz="0" iyz="0"/>
+    </inertial>
+  </link>
+  <joint name="left_wheel_joint" type="continuous">
+    <parent link="base_link"/>
+    <child link="left_wheel"/>
+    <origin xyz="0 0.2 -0.05" rpy="-1.5707 0 0"/>
+    <axis xyz="0 0 1"/>
+  </joint>
+  <link name="right_wheel">
+    <visual>
+      <geometry><cylinder radius="0.05" length="0.04"/></geometry>
+    </visual>
+    <collision>
+      <geometry><cylinder radius="0.05" length="0.04"/></geometry>
+    </collision>
+    <inertial>
+      <mass value="0.5"/>
+      <inertia ixx="0.001" iyy="0.001" izz="0.001" ixy="0" ixz="0" iyz="0"/>
+    </inertial>
+  </link>
+  <joint name="right_wheel_joint" type="continuous">
+    <parent link="base_link"/>
+    <child link="right_wheel"/>
+    <origin xyz="0 -0.2 -0.05" rpy="-1.5707 0 0"/>
+    <axis xyz="0 0 1"/>
+  </joint>
   <gazebo>
-    <plugin name ="diff_drive" filename="libgazebo_ros_diff_drive.so">
+    <plugin name="diff_drive" filename="libgazebo_ros_diff_drive.so">
       <left_joint>left_wheel_joint</left_joint>
       <right_joint>right_wheel_joint</right_joint>
@@ -17,8 +57,9 @@
       <publish_odom>true</publish_odom>
       <publish_odom_tf>true</publish_odom_tf>
-      <ros><remapping>cmd_vel:=/cmd_vel</remapping></ros>
+      <ros>
+        <remapping>cmd_vel:=/cmd_vel</remapping>
+      </ros>
     </plugin>
   </gazebo>
-  <!-- Simulated LiDAR: Publishes /scan -->
   <gazebo reference="base_link">
     <sensor name="laser" type="ray">
@@ -27,13 +68,20 @@
       <update_rate>10</update_rate>
       <ray>
-        <scan><horizontal>
-          <samples>360</samples>
-          <min_angle>-3.14159</min_angle>
-          <max_angle>3.14159</max_angle>
-        </horizontal></scan>
-        <range><min>0.1</min><max>10.0</max></range>
+        <scan>
+          <horizontal>
+            <samples>360</samples>
+            <min_angle>-3.14159</min_angle>
+            <max_angle>3.14159</max_angle>
+          </horizontal>
+        </scan>
+        <range>
+          <min>0.1</min>
+          <max>10.0</max>
+        </range>
       </ray>
       <plugin name="laser" filename="libgazebo_ros_ray_sensor.so">
-        <ros><remapping>~/out:=scan</remapping></ros>
+        <ros>
+          <remapping>~/out:=scan</remapping>
+        </ros>
         <output_type>sensor_msgs/LaserScan</output_type>
       </plugin>

Commit message: nandalal: Boustrophedon code been written and run by giving coordinatea instead of co-ordinate
FastAPI backend - sessions, zones, telemetry endpoints working

File: simulation/ros2_ws/src/cobot_sim/urdf/cobot.urdf.xacro (robot description, xacro)
@@ -1,7 +1,9 @@
 <?xml version="1.0"?>
 <robot name="cobot" xmlns:xacro="http://www.ros.org/wiki/xacro">
+  <!-- Base body -->
   <link name="base_link">
     <visual>
       <geometry><cylinder radius="0.2" length="0.15"/></geometry>
+      <material name="blue"><color rgba="0.0 0.0 0.8 1.0"/></material>
     </visual>
     <collision>
@@ -13,4 +15,5 @@
     </inertial>
   </link>
+  <!-- Left wheel -->
   <link name="left_wheel">
     <visual>
@@ -31,4 +34,5 @@
     <axis xyz="0 0 1"/>
   </joint>
+  <!-- Right wheel -->
   <link name="right_wheel">
     <visual>
@@ -49,5 +53,48 @@
     <axis xyz="0 0 1"/>
   </joint>
-<gazebo>
+  <!-- RealSense D435i camera link -->
+  <link name="camera_link">
+    <visual>
+      <geometry><box size="0.025 0.090 0.025"/></geometry>
+      <material name="black"><color rgba="0.0 0.0 0.0 1.0"/></material>
+    </visual>
+    <collision>
+      <geometry><box size="0.025 0.090 0.025"/></geometry>
+    </collision>
+    <inertial>
+      <mass value="0.072"/>
+      <inertia ixx="0.001" iyy="0.001" izz="0.001" ixy="0" ixz="0" iyz="0"/>
+    </inertial>
+  </link>
+  <joint name="camera_joint" type="fixed">
+    <parent link="base_link"/>
+    <child link="camera_link"/>
+    <origin xyz="0.2 0 0.05" rpy="0 0 0"/>
+  </joint>
+  <!-- Camera optical frame -->
+  <link name="camera_depth_frame"/>
+  <joint name="camera_depth_joint" type="fixed">
+    <parent link="camera_link"/>
+    <child link="camera_depth_frame"/>
+    <origin xyz="0 0 0" rpy="-1.5707 0 -1.5707"/>
+  </joint>
+  <!-- IMU link (MPU6050) -->
+  <link name="imu_link">
+    <visual>
+      <geometry><box size="0.02 0.02 0.005"/></geometry>
+      <material name="green"><color rgba="0.0 0.8 0.0 1.0"/></material>
+    </visual>
+    <inertial>
+      <mass value="0.01"/>
+      <inertia ixx="0.0001" iyy="0.0001" izz="0.0001" ixy="0" ixz="0" iyz="0"/>
+    </inertial>
+  </link>
+  <joint name="imu_joint" type="fixed">
+    <parent link="base_link"/>
+    <child link="imu_link"/>
+    <origin xyz="0 0 0.05" rpy="0 0 0"/>
+  </joint>
+  <!-- Diff-drive plugin -->
+  <gazebo>
     <plugin name="diff_drive" filename="libgazebo_ros_diff_drive.so">
       <left_joint>left_wheel_joint</left_joint>
@@ -57,13 +104,10 @@
       <publish_odom>true</publish_odom>
       <publish_odom_tf>true</publish_odom_tf>
-      <publish_wheel_tf>true</publish_wheel_tf>
-      <odometry_frame>odom</odometry_frame>
-      <robot_base_frame>base_link</robot_base_frame>
       <ros>
         <remapping>cmd_vel:=/cmd_vel</remapping>
-        <remapping>odom:=/odom</remapping>
       </ros>
     </plugin>
   </gazebo>
+  <!-- LiDAR sensor -->
   <gazebo reference="base_link">
     <sensor name="laser" type="ray">
@@ -79,16 +123,52 @@
           </horizontal>
         </scan>
-        <range>
-          <min>0.1</min>
-          <max>10.0</max>
-        </range>
+        <range><min>0.1</min><max>10.0</max></range>
       </ray>
       <plugin name="laser" filename="libgazebo_ros_ray_sensor.so">
-        <ros>
-          <remapping>~/out:=scan</remapping>
-        </ros>
+        <ros><remapping>~/out:=scan</remapping></ros>
         <output_type>sensor_msgs/LaserScan</output_type>
       </plugin>
     </sensor>
   </gazebo>
+  <!-- RealSense D435i depth camera plugin -->
+  <gazebo reference="camera_link">
+    <sensor name="depth_camera" type="depth">
+      <update_rate>30</update_rate>
+      <always_on>true</always_on>
+      <camera>
+        <horizontal_fov>1.5184</horizontal_fov>
+        <image>
+          <width>640</width>
+          <height>480</height>
+          <format>R8G8B8</format>
+        </image>
+        <clip><near>0.1</near><far>10.0</far></clip>
+      </camera>
+      <plugin name="depth_camera" filename="libgazebo_ros_camera.so">
+        <ros>
+          <remapping>~/image_raw:=/camera/color/image_raw</remapping>
+          <remapping>~/depth/image_raw:=/camera/depth/image_rect_raw</remapping>
+          <remapping>~/points:=/camera/depth/color/points</remapping>
+          <remapping>~/camera_info:=/camera/color/camera_info</remapping>
+        </ros>
+        <camera_name>camera</camera_name>
+        <frame_name>camera_depth_frame</frame_name>
+        <min_depth>0.1</min_depth>
+        <max_depth>10.0</max_depth>
+      </plugin>
+    </sensor>
+  </gazebo>
+  <!-- MPU6050 IMU plugin -->
+  <gazebo reference="imu_link">
+    <sensor name="imu_sensor" type="imu">
+      <always_on>true</always_on>
+      <update_rate>100</update_rate>
+      <plugin name="imu_plugin" filename="libgazebo_ros_imu_sensor.so">
+        <ros>
+          <remapping>~/out:=/imu/data</remapping>
+        </ros>
+        <initial_orientation_as_reference>false</initial_orientation_as_reference>
+      </plugin>
+    </sensor>
+  </gazebo>
 </robot>

Commit message: Entire code changed and version 1 Completed

File: simulation/ros2_ws/src/cobot_sim/urdf/cobot.urdf.xacro (robot description, xacro)
@@ -1,5 +1,5 @@
 <?xml version="1.0"?>
 <robot name="cobot" xmlns:xacro="http://www.ros.org/wiki/xacro">
-  <!-- Base body -->
+  <!-- ═══ BASE BODY ═══ -->
   <link name="base_link">
     <visual>
@@ -15,12 +15,8 @@
     </inertial>
   </link>
-  <!-- Left wheel -->
+  <!-- ═══ LEFT WHEEL ═══ -->
   <link name="left_wheel">
-    <visual>
-      <geometry><cylinder radius="0.05" length="0.04"/></geometry>
-    </visual>
-    <collision>
-      <geometry><cylinder radius="0.05" length="0.04"/></geometry>
-    </collision>
+    <visual><geometry><cylinder radius="0.05" length="0.04"/></geometry></visual>
+    <collision><geometry><cylinder radius="0.05" length="0.04"/></geometry></collision>
     <inertial>
       <mass value="0.5"/>
@@ -34,12 +30,8 @@
     <axis xyz="0 0 1"/>
   </joint>
-  <!-- Right wheel -->
+  <!-- ═══ RIGHT WHEEL ═══ -->
   <link name="right_wheel">
-    <visual>
-      <geometry><cylinder radius="0.05" length="0.04"/></geometry>
-    </visual>
-    <collision>
-      <geometry><cylinder radius="0.05" length="0.04"/></geometry>
-    </collision>
+    <visual><geometry><cylinder radius="0.05" length="0.04"/></geometry></visual>
+    <collision><geometry><cylinder radius="0.05" length="0.04"/></geometry></collision>
     <inertial>
       <mass value="0.5"/>
@@ -53,5 +45,5 @@
     <axis xyz="0 0 1"/>
   </joint>
-  <!-- RealSense D435i camera link -->
+  <!-- ═══ REALSENSE D435i CAMERA LINK ═══ -->
   <link name="camera_link">
     <visual>
@@ -59,7 +51,5 @@
       <material name="black"><color rgba="0.0 0.0 0.0 1.0"/></material>
     </visual>
-    <collision>
-      <geometry><box size="0.025 0.090 0.025"/></geometry>
-    </collision>
+    <collision><geometry><box size="0.025 0.090 0.025"/></geometry></collision>
     <inertial>
       <mass value="0.072"/>
@@ -79,5 +69,5 @@
     <origin xyz="0 0 0" rpy="-1.5707 0 -1.5707"/>
   </joint>
-  <!-- IMU link (MPU6050) -->
+  <!-- ═══ MPU6050 IMU LINK ═══ -->
   <link name="imu_link">
     <visual>
@@ -95,5 +85,5 @@
     <origin xyz="0 0 0.05" rpy="0 0 0"/>
   </joint>
-  <!-- Diff-drive plugin -->
+  <!-- ═══ DIFF DRIVE PLUGIN ═══ -->
   <gazebo>
     <plugin name="diff_drive" filename="libgazebo_ros_diff_drive.so">
@@ -104,10 +94,8 @@
       <publish_odom>true</publish_odom>
       <publish_odom_tf>true</publish_odom_tf>
-      <ros>
-        <remapping>cmd_vel:=/cmd_vel</remapping>
-      </ros>
+      <ros><remapping>cmd_vel:=/cmd_vel</remapping></ros>
     </plugin>
   </gazebo>
-  <!-- LiDAR sensor -->
+  <!-- ═══ LIDAR SENSOR ═══ -->
   <gazebo reference="base_link">
     <sensor name="laser" type="ray">
@@ -131,5 +119,5 @@
     </sensor>
   </gazebo>
-  <!-- RealSense D435i depth camera plugin -->
+  <!-- ═══ REALSENSE D435i DEPTH CAMERA PLUGIN ═══ -->
   <gazebo reference="camera_link">
     <sensor name="depth_camera" type="depth">
@@ -159,5 +147,5 @@
     </sensor>
   </gazebo>
-  <!-- MPU6050 IMU plugin -->
+  <!-- ═══ MPU6050 IMU PLUGIN ═══ -->
   <gazebo reference="imu_link">
     <sensor name="imu_sensor" type="imu">
@@ -165,7 +153,5 @@
       <update_rate>100</update_rate>
       <plugin name="imu_plugin" filename="libgazebo_ros_imu_sensor.so">
-        <ros>
-          <remapping>~/out:=/imu/data</remapping>
-        </ros>
+        <ros><remapping>~/out:=/imu/data</remapping></ros>
         <initial_orientation_as_reference>false</initial_orientation_as_reference>
       </plugin>
